Commit message: Add launch file and update xacro models for robot arm configuration

File: industrial_arm_description/xacro/gripper.xacro (robot description, xacro)
@@ -1,13 +1,15 @@
 <?xml version="1.0"?>
 <robot xmlns:xacro="http://www.ros.org/wiki/xacro">
-    <joint name="joint4" type="prismatic">
+    <joint name="joint4" type="revolute">
         <parent link="${frame_prefix}claw_support"/>
         <child link="${frame_prefix}gripper_right"/>
-        <origin xyz="0.01 -0.004 0.0" rpy="0 0 0"/> <axis xyz="0 1 0"/>
-        <limit lower="-0.015" upper="0.015" effort="5.0" velocity="1.0"/>
+        <origin xyz="0.18 -0.01 0.0" rpy="0 0 -${PI/2}"/>
+        <axis xyz="0 0 1"/>
+        <limit lower="-0.7" upper="0.0" effort="5.0" velocity="1.0"/>
     </joint>
     <link name="${frame_prefix}gripper_right">
         <visual>
-            <origin xyz="-0.1 0.5 -0.1" rpy="0 0 -${PI/2}"/> <geometry>
+            <origin xyz="-0.1 0.5 -0.1" rpy="0 0 -${PI/2}"/>
+            <geometry>
                 <mesh filename="package://industrial_arm_description/meshes/right_finger.STL" scale="${mesh_scale}"/>
             </geometry>
@@ -15,24 +17,25 @@
         </visual>
         <collision>
-            <origin xyz="0.01 0.01 0" rpy="0 0 0"/>
+            <origin xyz="0.01 0.02 0" rpy="0 0 0"/>
             <geometry>
-                <box size="0.01 0.03 0.02"/>
+                <box size="0.01 0.04 0.02"/>
             </geometry>
         </collision>
-        <xacro:inertial_box mass="0.02" x="0.01" y="0.03" z="0.02">
-            <origin xyz="0.01 0.01 0" rpy="0 0 0"/>
+        <xacro:inertial_box mass="0.02" x="0.01" y="0.04" z="0.02">
+            <origin xyz="0.01 0.02 0" rpy="0 0 0"/>
         </xacro:inertial_box>
     </link>
-    <joint name="gripper_left_joint" type="prismatic">
+    <joint name="gripper_left_joint" type="revolute">
         <parent link="${frame_prefix}claw_support"/>
         <child link="${frame_prefix}gripper_left"/>
-        <origin xyz="0.004 -0.004 0.0" rpy="0 0 0"/>
-        <axis xyz="0 1 0"/>
+        <origin xyz="0.18 0.165 -0.01" rpy="0 0 -${PI/2}"/>
+        <axis xyz="0 0 1"/>
         <mimic joint="joint4" multiplier="-1"/>
-        <limit lower="-0.015" upper="0.015" effort="5.0" velocity="1.0"/>
+        <limit lower="-0.7" upper="0.0" effort="5.0" velocity="1.0"/>
     </joint>
     <link name="${frame_prefix}gripper_left">
         <visual>
-            <origin xyz="-0.04 0.5 -0.1" rpy="0 0 -${PI/2}"/> <geometry>
+            <origin xyz="-0.04 0.5 -0.1" rpy="0 0 -${PI/2}"/>
+            <geometry>
                 <mesh filename="package://industrial_arm_description/meshes/left_finger.STL" scale="${mesh_scale}"/>
             </geometry>
@@ -40,11 +43,11 @@
         </visual>
         <collision>
-            <origin xyz="-0.01 0.01 0" rpy="0 0 0"/>
+            <origin xyz="-0.01 0.02 0" rpy="0 0 0"/>
             <geometry>
-                <box size="0.01 0.03 0.02"/>
+                <box size="0.01 0.04 0.02"/>
             </geometry>
         </collision>
-        <xacro:inertial_box mass="0.02" x="0.01" y="0.03" z="0.02">
-            <origin xyz="-0.01 0.01 0" rpy="0 0 0"/>
+        <xacro:inertial_box mass="0.02" x="0.01" y="0.04" z="0.02">
+            <origin xyz="-0.01 0.02 0" rpy="0 0 0"/>
         </xacro:inertial_box>
     </link>

File: industrial_arm_description/xacro/robot_core.xacro (robot description, xacro)
@@ -21,5 +21,5 @@
         <parent link="${frame_prefix}base_link"/>
         <child link="${frame_prefix}base_plate"/>
-        <origin xyz="0 0 0.0307" rpy="0 0 0"/> <axis xyz="0 0 1"/>
+        <origin xyz="0 0 0.307" rpy="0 0 0"/> <axis xyz="0 0 1"/>
         <limit lower="-${PI}" upper="${PI}" effort="10.0" velocity="2.5"/>
     </joint>
@@ -44,5 +44,5 @@
         <parent link="${frame_prefix}base_plate"/>
         <child link="${frame_prefix}forward_drive_arm"/>
-        <origin xyz="0 0.002 0.035" rpy="0 0 0"/> <axis xyz="0 1 0"/>
+        <origin xyz="0 0.02 0.35" rpy="0 0 0"/> <axis xyz="0 1 0"/>
         <limit lower="-${PI/2}" upper="${PI/2}" effort="15.0" velocity="2.0"/>
     </joint>
@@ -67,10 +67,10 @@
         <parent link="${frame_prefix}forward_drive_arm"/>
         <child link="${frame_prefix}horizontal_arm"/>
-        <origin xyz="0 0 0.080" rpy="0 0 0"/> <axis xyz="0 1 0"/>
+        <origin xyz="0 0 0.80" rpy="0 0 0"/> <axis xyz="0 1 0"/>
         <limit lower="-${PI/2}" upper="${PI/2}" effort="12.0" velocity="2.0"/>
     </joint>
     <link name="${frame_prefix}horizontal_arm">
         <visual>
-            <origin xyz="0.03 -0.4 -0.06" rpy="${PI/2} 0 ${PI/2}"/> <geometry>
+            <origin xyz="-0.03 -0.4 -0.06" rpy="${PI/2} 0 ${PI/2}"/> <geometry>
                 <mesh filename="package://industrial_arm_description/meshes/horizontal_arm.STL" scale="${mesh_scale}"/>
             </geometry>
@@ -90,8 +90,9 @@
         <parent link="${frame_prefix}horizontal_arm"/>
         <child link="${frame_prefix}claw_support"/>
-        <origin xyz="0.082 0 0" rpy="0 0 0"/> </joint>
+        <origin xyz="0.1 0.75 0" rpy="0 0 ${PI/2}"/>
+    </joint>
     <link name="${frame_prefix}claw_support">
         <visual>
-            <origin xyz="0 -0.05 -0.15" rpy="0 0 ${PI/2}"/> <geometry>
+            <origin xyz="0 -0.05 -0.15" rpy="0 0 ${PI*2}"/> <geometry>
                 <mesh filename="package://industrial_arm_description/meshes/claw_support.STL" scale="${mesh_scale}"/>
             </geometry>
