Commit message: Add industrial arm MoveIt configuration package
- Created .setup_assistant for MoveIt setup assistant configuration.
- Added CMakeLists.txt for build configuration.
- Introduced URDF and SRDF files for the industrial arm robot.
- Implemented ros2_control configuration in industrial_arm.ros2_control.xacro.
- Defined initial positions and joint limits in YAML files.
- Configured kinematics and MoveIt controllers for the industrial arm.
- Created launch files for demo, move group, RViz, and other functionalities.
- Established package.xml with dependencies and metadata for the industrial arm MoveIt configuration.

File: industrial_arm_description/xacro/robot_core.xacro (robot description, xacro)
@@ -44,5 +44,5 @@
         <parent link="${frame_prefix}base_plate"/>
         <child link="${frame_prefix}forward_drive_arm"/>
-        <origin xyz="0 0.02 0.35" rpy="0 0 0"/> <axis xyz="0 1 0"/>
+        <origin xyz="0 0.02 0.35" rpy="0 0 0"/> <axis xyz="1 0 0"/>
         <limit lower="-${PI/2}" upper="${PI/2}" effort="15.0" velocity="2.0"/>
     </joint>
@@ -67,5 +67,5 @@
         <parent link="${frame_prefix}forward_drive_arm"/>
         <child link="${frame_prefix}horizontal_arm"/>
-        <origin xyz="0 0 0.80" rpy="0 0 0"/> <axis xyz="0 1 0"/>
+        <origin xyz="0 0 0.80" rpy="0 0 0"/> <axis xyz="1 0 0"/>
         <limit lower="-${PI/2}" upper="${PI/2}" effort="12.0" velocity="2.0"/>
     </joint>
